File: spacecadet/USB-C.kicad_sch (KiCad schematic)
At the start: 4 parts

Commit message: First rev fully routed. (3D for keycaps is not redistibutable)
Parts:
- removed ESD1: PRTR5V0U2X, Keyboardio:PRTR5V0U2X, symbol Keyboard-symbols:Power_Protection_PRTR5V0U2X-prtr5v0u2x
- removed R6, R7: 5.1K, Resistor_SMD:R_0603_1608Metric, symbol Device:R
- removed USB1: USB_C_Receptacle, Keyboardio:USB-TYPE-C-MIDMOUNT, symbol Keyboard-symbols:USB_C_Receptacle-usb_c_receptacle
Connections:
- no-connect marks 10 -> 0
Other:
- removed sheet USB Support
- note removed: "USB ESD Protection"
- note removed: "USB Support Circuitry"
- note removed: "USB Type C Mid Connector"
