File: spacecadet/Key_Matrix.kicad_sch (KiCad schematic)
At the start: 200 parts

Commit message: First rev fully routed. (3D for keycaps is not redistibutable)
Parts:
- SW_95: value (none) -> ~
Connections:
- net COL23 is gone; now on net COL20: D_SW_33.2 (A), D_SW_54.2 (A), D_SW_91.2 (A)
- net COL10: now also D_SW_23.2 (A), D_SW_44.2 (A), D_SW_64.2 (A), D_SW_82.2 (A); no longer D_SW_22.2 (A), D_SW_43.2 (A), D_SW_6.2 (A), D_SW_63.2 (A), D_SW_81.2 (A), D_SW_95.2 (A)
- net COL11: now also D_SW_24.2 (A), D_SW_45.2 (A), D_SW_65.2 (A), D_SW_7.2 (A), D_SW_83.2 (A); no longer D_SW_23.2 (A), D_SW_44.2 (A), D_SW_64.2 (A), D_SW_82.2 (A)
- net COL12: now also D_SW_25.2 (A), D_SW_46.2 (A), D_SW_66.2 (A), D_SW_84.2 (A); no longer D_SW_24.2 (A), D_SW_45.2 (A), D_SW_65.2 (A), D_SW_7.2 (A), D_SW_83.2 (A)
- net COL13: now also D_SW_26.2 (A), D_SW_47.2 (A), D_SW_67.2 (A), D_SW_8.2 (A), D_SW_85.2 (A); no longer D_SW_25.2 (A), D_SW_46.2 (A), D_SW_66.2 (A), D_SW_84.2 (A)
- net COL14: now also D_SW_27.2 (A), D_SW_48.2 (A), D_SW_68.2 (A), D_SW_86.2 (A); no longer D_SW_26.2 (A), D_SW_47.2 (A), D_SW_67.2 (A), D_SW_8.2 (A), D_SW_85.2 (A)
- net COL15: now also D_SW_28.2 (A), D_SW_49.2 (A), D_SW_69.2 (A), D_SW_87.2 (A), D_SW_9.2 (A), D_SW_96.2 (A); no longer D_SW_27.2 (A), D_SW_48.2 (A), D_SW_68.2 (A), D_SW_86.2 (A)
- net COL16: now also D_SW_29.2 (A), D_SW_50.2 (A); no longer D_SW_28.2 (A), D_SW_49.2 (A), D_SW_87.2 (A), D_SW_9.2 (A), D_SW_96.2 (A)
- net COL17: now also D_SW_10.2 (A), D_SW_30.2 (A), D_SW_51.2 (A), D_SW_70.2 (A), D_SW_88.2 (A), D_SW_97.2 (A); no longer D_SW_50.2 (A), D_SW_69.2 (A)
- net COL18: now also D_SW_11.2 (A), D_SW_31.2 (A), D_SW_52.2 (A), D_SW_71.2 (A), D_SW_89.2 (A), D_SW_98.2 (A); no longer D_SW_10.2 (A), D_SW_29.2 (A), D_SW_51.2 (A), D_SW_70.2 (A), D_SW_88.2 (A)
- net COL19: now also D_SW_12.2 (A), D_SW_32.2 (A), D_SW_53.2 (A), D_SW_90.2 (A), D_SW_99.2 (A); no longer D_SW_30.2 (A), D_SW_97.2 (A)
- net COL2: now also D_SW_94.2 (A)
- net COL20: now also D_SW_72.2 (A); no longer D_SW_11.2 (A), D_SW_31.2 (A), D_SW_52.2 (A), D_SW_71.2 (A), D_SW_89.2 (A)
- net COL3: now also D_SW_100.2 (A), D_SW_16.2 (A), D_SW_3.2 (A), D_SW_37.2 (A), D_SW_57.2 (A), D_SW_76.2 (A); no longer D_SW_94.2 (A)
- net COL4: now also D_SW_17.2 (A), D_SW_38.2 (A), D_SW_58.2 (A); no longer D_SW_100.2 (A), D_SW_16.2 (A), D_SW_3.2 (A), D_SW_37.2 (A), D_SW_57.2 (A), D_SW_76.2 (A)
- net COL5: now also D_SW_18.2 (A), D_SW_39.2 (A), D_SW_4.2 (A), D_SW_59.2 (A), D_SW_77.2 (A); no longer D_SW_17.2 (A), D_SW_38.2 (A), D_SW_58.2 (A)
- net COL6: now also D_SW_19.2 (A), D_SW_40.2 (A), D_SW_60.2 (A), D_SW_78.2 (A); no longer D_SW_18.2 (A), D_SW_39.2 (A), D_SW_4.2 (A), D_SW_59.2 (A), D_SW_77.2 (A)
- net COL7: now also D_SW_20.2 (A), D_SW_41.2 (A), D_SW_5.2 (A), D_SW_61.2 (A), D_SW_79.2 (A); no longer D_SW_19.2 (A), D_SW_40.2 (A), D_SW_60.2 (A), D_SW_78.2 (A)
- net COL8: now also D_SW_21.2 (A), D_SW_42.2 (A), D_SW_62.2 (A), D_SW_80.2 (A); no longer D_SW_20.2 (A), D_SW_41.2 (A), D_SW_5.2 (A), D_SW_61.2 (A), D_SW_79.2 (A)
- net COL9: now also D_SW_22.2 (A), D_SW_43.2 (A), D_SW_6.2 (A), D_SW_63.2 (A), D_SW_81.2 (A), D_SW_95.2 (A); no longer D_SW_21.2 (A), D_SW_42.2 (A), D_SW_62.2 (A), D_SW_80.2 (A)
- removed net COL21: D_SW_90.2 (A), D_SW_98.2 (A)
- removed net COL22: D_SW_12.2 (A), D_SW_32.2 (A), D_SW_53.2 (A), D_SW_72.2 (A), D_SW_99.2 (A)
Other:
- moved on the sheet: D_SW_1, D_SW_10, D_SW_100, D_SW_11, D_SW_12, D_SW_13, D_SW_14, D_SW_15, D_SW_16, D_SW_17, D_SW_18, D_SW_19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

Commit message: Add some mounting holes
Parts:
- added STAB1: Stabilizer_Cherry_MX_8.00u, Mounting_Keyboard_Stabilizer:Stabilizer_Cherry_MX_8.00u, symbol Mechanical:MountingHole
- SW_1, SW_10, SW_11, SW_12, SW_15, SW_2, SW_3, SW_31, SW_36, SW_4, SW_5, SW_52, SW_55, SW_56, SW_6, SW_69, SW_7, SW_71, SW_72, SW_8, SW_9: footprint Keyboardio:MX-KailhClip-1.00u -> Keyboardio:MX-KailhClip-2u-no-top-ring
- SW_100, SW_57, SW_96: footprint Keyboardio:MX-KailhClip-1.00u -> Keyboardio:MX-KailhClip-1.75u-no-top-ring
- SW_13, SW_14, SW_16, SW_17, SW_18, SW_19, SW_20, SW_21, SW_22, SW_23, SW_24, SW_25, SW_26, SW_29, SW_30, SW_32, SW_33, SW_34, SW_35, SW_38, SW_39, SW_40, SW_41, SW_42, SW_43, SW_44, SW_45, SW_46, SW_47, SW_48, SW_49, SW_50, SW_53, SW_54, SW_58, SW_59, SW_60, SW_61, SW_62, SW_63, SW_64, SW_65, SW_66, SW_67, SW_68, SW_73, SW_77, SW_78, SW_79, SW_80, SW_81, SW_82, SW_83, SW_84, SW_85, SW_86, SW_91: footprint Keyboardio:MX-KailhClip-1.00u -> Keyboardio:MX-KailhClip-1.00u-no-top-ring
- SW_27, SW_28, SW_37, SW_51, SW_74, SW_75, SW_88, SW_89, SW_90, SW_92, SW_93, SW_94, SW_97, SW_98, SW_99: footprint Keyboardio:MX-KailhClip-1.00u -> Keyboardio:MX-KailhClip-1.5u-no-top-ring
- SW_70: footprint Keyboardio:MX-KailhClip-1.00u -> Keyboardio:MX-KailhClip-1.25u-no-top-ring
- SW_76, SW_87: footprint Keyboardio:MX-KailhClip-1.00u -> Keyboardio:MX-KailhClip-2.25u-no-top-ring
- SW_95: footprint Keyboardio:MX-KailhClip-1.00u -> Keyboardio:MX-KailhClip-7u-no-top-ring

Commit message: Fix diode footprint to Keyboardio's standard. Remove some key labels that broke the kicad-jlc integration
Parts:
- D_SW_1, D_SW_10, D_SW_100, D_SW_11, D_SW_12, D_SW_13, D_SW_14, D_SW_15, D_SW_16, D_SW_17, D_SW_18, D_SW_19, D_SW_2, D_SW_20, D_SW_21, D_SW_22, D_SW_23, D_SW_24, D_SW_25, D_SW_26, D_SW_27, D_SW_28, D_SW_29, D_SW_3, D_SW_30, D_SW_31, D_SW_32, D_SW_33, D_SW_34, D_SW_35, D_SW_36, D_SW_37, D_SW_38, D_SW_39, D_SW_4, D_SW_40, D_SW_41, D_SW_42, D_SW_43, D_SW_44, D_SW_45, D_SW_46, D_SW_47, D_SW_48, D_SW_49, D_SW_5, D_SW_50, D_SW_51, D_SW_52, D_SW_53, D_SW_54, D_SW_55, D_SW_56, D_SW_57, D_SW_58, D_SW_59, D_SW_6, D_SW_60, D_SW_61, D_SW_62, D_SW_63, D_SW_64, D_SW_65, D_SW_66, D_SW_67, D_SW_68, D_SW_69, D_SW_7, D_SW_70, D_SW_71, D_SW_72, D_SW_73, D_SW_74, D_SW_75, D_SW_76, D_SW_77, D_SW_78, D_SW_79, D_SW_8, D_SW_80, D_SW_81, D_SW_82, D_SW_83, D_SW_84, D_SW_85, D_SW_86, D_SW_87, D_SW_88, D_SW_89, D_SW_9, D_SW_90, D_SW_91, D_SW_92, D_SW_93, D_SW_94, D_SW_95, D_SW_96, D_SW_97, D_SW_98, D_SW_99: footprint Diode_SMD:D_SOD-123 -> Keyboardio:D_SOD-123-Keyboardio
- SW_4: value OVER<BR>STRIKE -> OVERSTRIKE
