File: spacecadet/spacecadet.kicad_sch (KiCad schematic)
At the start: 0 parts

Commit message: First rev fully routed. (3D for keycaps is not redistibutable)
Parts:
- added C1, C2: 1uF, Capacitor_SMD:C_0603_1608Metric, symbol Device:C
- added C12: 10nF 100V, Capacitor_SMD:C_0805_2012Metric, symbol model100-left-rescue:CSMALL
- added C13, C14: 27pF DNP, Capacitor_SMD:C_0603_1608Metric, symbol model100-left-rescue:CSMALL
- added C15, C16: 4.7uF 16V X7R, Capacitor_SMD:C_1210_3225Metric, symbol model100-left-rescue:CSMALL
- added C5, C6, C7, C8, C9: 1µF ±20% 10V Ceramic Capacitor X5R 0603 (1608 Met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, Capacitor_SMD:C_0603_1608Metric, symbol modela-rescue:CSMALL
- added D1, D2, D3: WS2812B, LED_SMD:LED_WS2812B_PLCC4_5.0x5.0mm_P3.2mm, symbol LED:WS2812B
- added F1: PTC RESET FUSE 6V 750MA 1206, Fuse:Fuse_1206_3216Metric, symbol Device:Polyfuse
- added J1: Conn_01x05_Male, Connector_PinHeader_2.54mm:PinHeader_1x05_P2.54mm_Vertical, symbol Connector:Conn_01x05_Male
- added JP1: SolderJumper_2_Open, Jumper:SolderJumper-2_P1.3mm_Bridged_RoundedPad1.0x1.5mm, symbol Jumper:SolderJumper_2_Open
- added L2: FERRITE BEAD 390 OHM 1206 1LN, Capacitor_SMD:C_1206_3216Metric, symbol model100-left-rescue:INDUCTOR_SMALL
- added R1, R2, R4, R7, R8: 10K, Resistor_SMD:R_0603_1608Metric, symbol Device:R
- added R3: 300R, Resistor_SMD:R_0603_1608Metric, symbol Device:R
- added R31: 500K, Resistor_SMD:R_0603_1608Metric, symbol model100-left-rescue:R
- added R32, R33: 22R, Resistor_SMD:R_0603_1608Metric, symbol model100-left-rescue:R
- added R34, R35: 5.1K 1%, Resistor_SMD:R_0603_1608Metric, symbol model100-left-rescue:R
- added R5: 1.5k, Resistor_SMD:R_0603_1608Metric, symbol Device:R
- added R6: 10K, Resistor_SMD:R_0603_1608Metric, symbol modela-rescue:R
- added RV1, RV2: V5.5MLA0603NH, Resistor_SMD:R_0603_1608Metric, symbol Device:Varistor
- added SW1: SW_PUSH, Button_Switch_SMD:SW_SPST_TL3342, symbol modela-rescue:SW_PUSH
- added T2: USBD-, Keyboardio:Labeled_TestPoint_Pad_2mm, symbol test-point:TST
- added T3: USBD+, Keyboardio:Labeled_TestPoint_Pad_2mm, symbol test-point:TST
- added U1: MIC5504-3.3YM5-TR, Package_TO_SOT_SMD:SOT-23-5, symbol modela-rescue:MIC5504-3.3YM5-TR
- added U2: GD32F303CGT6, Package_QFP:LQFP-48_7x7mm_P0.5mm, symbol modela-rescue:GD32F303CGTx
- added U4: SRV05-4HTG, Package_TO_SOT_SMD:SOT-23-6, symbol model100-left-rescue:SRV05
- added USB1: USB - C USB 3.1 (USB 3.1 Gen 2, Superspeed+) Rece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, Connector_USB:USB_C_Receptacle_HRO_TYPE-C-31-M-12, symbol model100-left-rescue:Type-C_midmount
Connections:
- new net: R35.1, USB1.A5 (CC1)
- new net: R34.1, USB1.B5 (CC2)
- new net: D2.2 (DOUT), D3.4 (DIN)
- new net: D1.2 (DOUT), D2.4 (DIN)
- new net: D1.4 (DIN), R3.2
- new net: R1.1, U1.3 (EN)
- new net +3V3: C2.1, C5.1, C6.1, C7.1, C8.1, D1.1 (VDD), D2.1 (VDD), D3.1 (VDD), J1.2 (Pin_2), JP1.1 (A), R6.2, R7.2, R8.2, U1.5 (VOUT), U2.1 (VBAT), U2.24 (VDD), U2.36 (VDD), U2.48 (VDD), U2.9 (VDDA)
- new net +5V: C1.1, C16.1, L2.2, R1.2, U1.1 (VIN)
- new net BOOT0: JP1.2 (B), U2.44 (BOOT0)
- new net COL0: U2.19 (PB1)
- new net COL1: U2.18 (PB0)
- new net COL10: U2.6 (OSC_OUT(PD1))
- new net COL11: U2.5 (OSC_IN(PD0))
- new net COL12: U2.4 (PC15)
- new net COL13: U2.3 (PC14)
- new net COL14: U2.2 (PC13)
- new net COL15: U2.30 (PA9)
- new net COL16: U2.31 (PA10)
- new net COL17: U2.45 (PB8)
- new net COL18: U2.43 (PB7)
- new net COL19: U2.42 (PB6)
- new net COL2: U2.17 (PA7)
- new net COL20: U2.41 (PB5)
- new net COL21: U2.46 (PB9)
- new net COL3: U2.16 (PA6)
- new net COL4: U2.15 (PA5)
- new net COL5: U2.14 (PA4)
- new net COL6: U2.13 (PA3)
- new net COL7: U2.12 (PA2)
- new net COL8: U2.11 (PA1)
- new net COL9: U2.10 (PA0)
- new net GND: C1.2, C12.2, C13.2, C14.2, C15.2, C16.2, C2.2, C5.2, C6.2, C7.2, C8.2, C9.2, D1.3 (VSS), D2.3 (VSS), D3.3 (VSS), J1.5 (Pin_5), R2.2, R31.2, R34.2, R35.2, R4.2, RV2.1, SW1.1, U1.2 (GND), U2.23 (VSS), U2.35 (VSS), U2.47 (VSS), U2.8 (VSSA), U4.2 (GND), USB1.A1 (GND), USB1.A12 (GND), USB1.B1 (GND), USB1.B12 (GND)
- new net JTCLK/SWCLK: J1.4 (Pin_4), R4.1, U2.37 (PA14)
- new net JTDI: U2.38 (PA15)
- new net JTDO: U2.39 (PB3)
- new net JTMS/SWDIO: J1.3 (Pin_3), R7.1, U2.34 (PA13)
- new net MOSI: R3.1
- new net PB2: R2.1, U2.20 (PB2(BOOT1))
- new net RD+: R33.2, U2.33 (PA12(USBDP))
- new net RD-: R32.2, U2.32 (PA11(USBDM))
- new net RESET_MCU: C9.1, R6.1, SW1.2, U2.7 (NRST)
- new net ROW0: U2.28 (PB15)
- new net ROW1: U2.27 (PB14)
- new net ROW2: U2.26 (PB13)
- new net ROW3: U2.25 (PB12)
- new net ROW4: U2.22 (PB11)
- new net ROW5: U2.21 (PB10)
- new net USBD+: C13.1, R33.1, R5.2, T3.1, U4.1 (IO_1), U4.3 (IO_2), USB1.A6 (D+), USB1.B6 (D+)
- new net USBD-: C14.1, R32.1, T2.1, U4.4 (IO_3), U4.6 (IO_4), USB1.A7 (D-), USB1.B7 (D-)
- new net USBDP_PULLUP: R5.1, U2.29 (PA8)
- new net USBSHIELD: C12.1, R31.1, RV1.2, RV2.2, USB1.S1 (Shield)
- new net USBVBUS: F1.2, RV1.1, USB1.A4 (VBUS), USB1.A9 (VBUS), USB1.B4 (VBUS), USB1.B9 (VBUS)
- new net VBUS_FUSED: C15.1, F1.1, L2.1, U4.5 (VCC)
- new net ~JTRST~: J1.1 (Pin_1), R8.1, U2.40 (PB4)
- no-connect marks 0 -> 10
Other:
- removed sheet MCU-ATmega32u4
- removed sheet USB-C
- note added: "ESD Protection"
- note added: "Filtering"
- note added: "For a full pin description, please refer to pgs. 38 to 40 in the datasheet: https://www.gigadevice.com/datasheet/gd32f303xxxx-datasheet/ Here you will find each pin definition and peripheral relation. Note: Most alternate/primary pin functions have been reserved."
- note added: "MCU Programming"
- note added: "Optional slew rate limiting if required for EMI (probably not required)"
- note added: "Overvoltage Protection"
- note added: "Place close to 2xVCC, 2x AVCC pins."
- note added: "Primary Microcontroller"
- note added: "Used for programming bootloader but can still be used as GPIO."
- note added: "Varistors for overvoltage protection per https://m.littelfuse.com/~/media/electronics_technical/application_notes/usb/ littelfuse_why_does_usb_2_0_need_circuit_protection_application_note.pdf"
- note added: "Wire 0,0 to the main MCU so we can use it to force reprogramming"
- note removed: "Microcontroller"
- note removed: "USB Connector"

Commit message: Fix boot0 jumper design
Parts:
- added R9: 10K, Resistor_SMD:R_0603_1608Metric, symbol Device:R
- JP1: footprint Jumper:SolderJumper-2_P1.3mm_Bridged_RoundedPad1.0x1.5mm -> Jumper:SolderJumper-3_P1.3mm_Bridged12_Pad1.0x1.5mm; symbol Jumper:SolderJumper_2_Open -> Jumper:SolderJumper_3_Bridged12; now in the parts list
Connections:
- net +3V3: now also JP1.3 (B); no longer JP1.1 (A)
- net BOOT0: now also R9.2; no longer JP1.2 (B)
- net GND: now also JP1.2 (C)
- new net: JP1.1 (A), R9.1
Other:
- note removed: "MCU Programming"
- moved on the sheet: C9, D1, D2, D3, J1, R3, R4, R6, R7, R8, SW1

Commit message: Correct wiring of BOOT0 jumper
Connections:
- net GND: now also JP1.1 (A); no longer JP1.2 (C)
- net at R9.1: now also JP1.2 (C); no longer JP1.1 (A)
Other:
- moved on the sheet: JP1
Changed lines of the file:
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@@
     (stroke (width 0) (type default) (color 0 0 0 0))
   )
-  (wire (pts (xy 414.02 49.7332) (xy 414.02 50.8))
+  (wire (pts (xy 414.02 49.53) (xy 414.02 50.8))
     (stroke (width 0) (type default) (color 0 0 0 0))
   )
@@
     (stroke (width 0) (type solid) (color 0 0 0 0))
   )
-  (wire (pts (xy 417.83 44.6532) (xy 418.6936 44.6532))
+  (wire (pts (xy 408.94 45.72) (xy 408.94 48.26))
     (stroke (width 0) (type default) (color 0 0 0 0))
   )
@@
     (pin "2")
   )
-  (symbol (lib_id "Jumper:SolderJumper_3_Bridged12") (at 414.02 44.6532 90) (unit 1)
-    (in_bom yes) (on_board yes)
-    (property "Reference" "JP1" (id 0) (at 412.2928 44.6532 90)
-      (effects (font (size 1.27 1.27)) (justify left))
-    )
-    (property "Value" "SolderJumper_2_Open" (id 1) (at 412.2928 43.5102 90)
+  (symbol (lib_id "Jumper:SolderJumper_3_Bridged12") (at 414.02 45.72 0) (unit 1)
+    (in_bom yes) (on_board yes)
+    (property "Reference" "JP1" (id 0) (at 414.02 43.9928 90)
+      (effects (font (size 1.27 1.27)) (justify left))
+    )
+    (property "Value" "SolderJumper_2_Open" (id 1) (at 415.163 43.9928 90)
       (effects (font (size 1.27 1.27)) (justify left) hide)
     )
-    (property "Footprint" "Jumper:SolderJumper-3_P1.3mm_Bridged12_Pad1.0x1.5mm" (id 2) (at 414.02 44.6532 0)
-      (effects (font (size 1.27 1.27)) hide)
-    )
-    (property "Datasheet" "~" (id 3) (at 414.02 44.6532 0)
-      (effects (font (size 1.27 1.27)) hide)
-    )
-    (property "Config" "DNP" (id 4) (at 414.02 44.6532 0)
+    (property "Footprint" "Jumper:SolderJumper-3_P1.3mm_Bridged12_Pad1.0x1.5mm" (id 2) (at 414.02 45.72 0)
+      (effects (font (size 1.27 1.27)) hide)
+    )
+    (property "Datasheet" "~" (id 3) (at 414.02 45.72 0)
+      (effects (font (size 1.27 1.27)) hide)
+    )
+    (property "Config" "DNP" (id 4) (at 414.02 45.72 0)
       (effects (font (size 1.27 1.27)) hide)
     )
@@
     (pin "1")
   )
-  (symbol (lib_id "power:+3.3V") (at 414.02 39.5732 0) (unit 1)
-    (in_bom yes) (on_board yes)
-    (property "Reference" "#PWR07" (id 0) (at 414.02 43.3832 0)
-      (effects (font (size 1.27 1.27)) hide)
-    )
-    (property "Value" "+3.3V" (id 1) (at 414.401 35.179 0))
-    (property "Footprint" "" (id 2) (at 414.02 39.5732 0)
-      (effects (font (size 1.27 1.27)) hide)
-    )
-    (property "Datasheet" "" (id 3) (at 414.02 39.5732 0)
+  (symbol (lib_id "power:+3.3V") (at 419.1 45.72 0) (unit 1)
+    (in_bom yes) (on_board yes)
+    (property "Reference" "#PWR07" (id 0) (at 419.1 49.53 0)
+      (effects (font (size 1.27 1.27)) hide)
+    )
+    (property "Value" "+3.3V" (id 1) (at 419.481 41.3258 0))
+    (property "Footprint" "" (id 2) (at 419.1 45.72 0)
+      (effects (font (size 1.27 1.27)) hide)
+    )
+    (property "Datasheet" "" (id 3) (at 419.1 45.72 0)
       (effects (font (size 1.27 1.27)) hide)
     )
@@
     (pin "1")
   )
-  (symbol (lib_id "model100-left-rescue:GND") (at 418.6936 44.6532 90) (unit 1)
+  (symbol (lib_id "model100-left-rescue:GND") (at 408.94 48.26 0) (unit 1)
     (in_bom yes) (on_board yes) (fields_autoplaced)
-    (property "Reference" "#PWR0101" (id 0) (at 418.6936 44.6532 0)
-      (effects (font (size 0.762 0.762)) hide)
-    )
-    (property "Value" "GND" (id 1) (at 420.4716 44.6532 0)
-      (effects (font (size 0.762 0.762)) hide)
-    )
-    (property "Footprint" "" (id 2) (at 418.6936 44.6532 0)
-      (effects (font (size 1.524 1.524)))
-    )
-    (property "Datasheet" "" (id 3) (at 418.6936 44.6532 0)
-      (effects (font (size 1.524 1.524)))
-    )
+    (property "Reference" "#PWR0101" (id 0) (at 408.94 48.26 0)
+      (effects (font (size 0.762 0.762)) hide)
+    )
+    (property "Value" "GND" (id 1) (at 408.94 50.038 0)
+      (effects (font (size 0.762 0.762)) hide)
+    )
+    (property "Footprint" "" (id 2) (at 408.94 48.26 0)
+      (effects (font (size 1.524 1.524)))
+    )
+    (property "Datasheet" "" (id 3) (at 408.94 48.26 0)
+      (effects (font (size 1.524 1.524)))
+    )
